File: pcb_blheli_s.kicad_pcb (KiCad board)
At the start: 2 copper layers, 29.2 x 13 mm, 23 parts, among them IC1 EFM8BB21F16G-C-QFN20, IC2 REG113NA-3.3_250, J1 Conn_01x03_Pin, J2 Conn_01x04_Pin, J3 Conn_01x03_Socket, Q1 DMN2058U, Q2 DMN2058U, Q3 DMN2058U, Q4 DMN2058U, Q5 DMN2058U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

Commit message: Finished gerber
Parts:
- moved J3 1.30 mm to (140.2, 102.0)
- moved Q6 1.30 mm to (136.8, 107.4)
- moved Q4 1.22 mm to (136.8, 103.5)
- moved Q2 1.20 mm to (136.8, 99.6)
- moved Q5 1.03 mm to (133.3, 107.4)
- moved Q3 0.92 mm to (133.3, 103.5)
- moved Q1 0.90 mm to (133.3, 99.6)
- moved C2 0.25 mm to (116.0, 103.2)
- moved R7 0.21 mm to (128.8, 103.7)
- moved R8 0.21 mm to (128.8, 107.2)
- moved R3 0.20 mm to (128.8, 100.2)
- moved R4 0.20 mm to (128.8, 98.5)
- moved R5 0.20 mm to (128.8, 102.0)
- moved R6 0.20 mm to (128.8, 105.5)
Routing:
- net VDC: track 46.6 -> 44.5 mm
- net Net-(J3-Pin_1): track 16.0 -> 14.2 mm
- net /COM_A: track 12.4 -> 11.0 mm
- net /PWM_C: track 12.2 -> 11.1 mm
- net /PWM_A: track 7.93 -> 6.95 mm
- net /PWM_B: track 10.1 -> 9.12 mm
- net /COM_C: track 17.8 -> 16.9 mm
- net Net-(J3-Pin_3): track 17.5 -> 16.6 mm
- net /COM_B: track 14.9 -> 14.0 mm
- net Net-(J3-Pin_2): track 16.3 -> 15.6 mm
Other:
- board size 29.2 x 13 mm -> 28 x 13 mm

Commit message: Updated schematics
Parts:
- added J4: Conn_01x03_Pin, Connector_PinHeader_2.00mm:PinHeader_1x03_P2.00mm_Vertical, F.Cu at (120.7, 98.1)
- added R10: 2K2, Resistor_SMD:R_0603_1608Metric, B.Cu at (130.1, 104.9)
- added R11: 2K2, Resistor_SMD:R_0603_1608Metric, B.Cu at (130.1, 106.6)
- added R9: 2K2, Resistor_SMD:R_0603_1608Metric, B.Cu at (130.1, 98.5)
- J3: footprint Connector_PinHeader_1.27mm:PinHeader_1x03_P1.27mm_Vertical -> Connector_PinHeader_2.00mm:PinHeader_1x03_P2.00mm_Vertical
- moved C3 2.21 mm to (119.1, 107.8)
- moved C4 2.01 mm to (119.6, 100.4)
- moved R2 1.94 mm to (116.6, 100.4)
- moved C1 1.77 mm to (119.6, 101.9)
- moved J2 1.71 mm to (121.9, 108.6)
- moved IC2 1.51 mm to (118.8, 104.5)
- moved R4 1.39 mm to (130.1, 99.1)
- moved R3 1.30 mm to (130.1, 100.6)
- moved R7 1.25 mm to (130.1, 103.6)
- moved R8 1.25 mm to (130.1, 107.1)
- moved R5 1.25 mm to (130.1, 102.1)
- moved R6 1.25 mm to (130.1, 105.5)
- moved J3 0.92 mm to (140.0, 101.1)
- moved C2 0.86 mm to (115.9, 104.1)
- moved R1 0.60 mm to (122.4, 106.2)
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Connections:
- net Net-(IC1-P0.5) renamed /RX0
- IC1 pad 18: /BL_TX2 -> /TX0
- Q1 pad 2: GND -> Net-(J3-Pin_1)
- Q1 pad 3: Net-(J3-Pin_1) -> VDC
- Q2 pad 2: VDC -> GND
- Q3 pad 2: GND -> Net-(J3-Pin_2)
- Q3 pad 3: Net-(J3-Pin_2) -> VDC
- Q4 pad 2: VDC -> GND
- Q5 pad 2: GND -> Net-(J3-Pin_3)
- Q5 pad 3: Net-(J3-Pin_3) -> VDC
- Q6 pad 2: VDC -> GND
Routing:
- net /TX0: track 0.00 -> 6.15 mm, vias 0 -> 1
- net VDC: track 44.5 -> 39.0 mm
- net /RX0: track 9.14 -> 12.2 mm, vias 2 -> 1
- net /MUX_C: track 12.2 -> 14.5 mm, vias 2 -> 3
- net /MUX_B: track 9.72 -> 11.8 mm, vias 2 -> 3
- net /MUX_A: track 5.85 -> 7.95 mm, vias 0 -> 1
- net /COM_C: track 16.9 -> 14.9 mm, vias 0 -> 2
- net Net-(J3-Pin_2): track 15.6 -> 14.1 mm
- net /RC_IN: track 3.28 -> 1.92 mm
- net /PWM_B: track 9.12 -> 7.90 mm
- net GND: track 8.65 -> 7.50 mm, vias 4 -> 10
- net /COMP_COM: track 9.16 -> 10.1 mm
- net Net-(J3-Pin_1): track 14.2 -> 13.4 mm
- net +3.3V: track 13.9 -> 14.8 mm
- net /COM_B: track 14.0 -> 14.6 mm
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Other:
- board size 28 x 13 mm -> 28 x 13.5 mm

Commit message: Updated gerber
Parts:
- moved J1 0.51 mm to (113.3, 103.3)
- moved C3 0.50 mm to (119.1, 107.3)
- moved Q5 0.40 mm to (133.3, 107.6)
- moved Q6 0.40 mm to (136.8, 107.6)
- moved Q1 0.40 mm to (133.3, 99.7)
- moved Q2 0.40 mm to (136.8, 99.7)
- moved Q3 0.40 mm to (133.3, 103.7)
- moved Q4 0.40 mm to (136.8, 103.7)
- moved IC1 0.10 mm to (124.6, 102.4)
Routing:
- net /COM_C: track 14.9 -> 15.8 mm, vias 2 -> 0
- net Net-(J3-Pin_3): track 16.1 -> 15.5 mm
- net Net-(IC2-NR): track 2.42 -> 1.92 mm
- net /PWM_C: track 10.7 -> 10.4 mm, vias 2 -> 0
- net GND: track 7.50 -> 7.64 mm, vias 10 -> 15
Other:
- board text added: "BLHeli_S 1S REV2"
- board text added: "G CK 3V D"
- board text added: "G R T"

Commit message: Ordered rev2
Parts:
- Q2, Q4, Q6: value DMN2058U -> IRLML2244TRPBF; footprint Package_TO_SOT_SMD:SOT-23 -> footprint_blheli:SOT95P237X112-3N
- moved R11 0.58 mm to (129.8, 107.1)
- moved J3 0.14 mm to (140.1, 101.0)
- moved Q6 0.05 mm to (136.8, 107.7)
Connections:
- J2 pad 2: /C2CK -> +3.3V
- J2 pad 3: +3.3V -> /C2CK
- Q1 pad 2: Net-(J3-Pin_1) -> GND
- Q1 pad 3: VDC -> Net-(J3-Pin_1)
- Q2 pad 2: GND -> VDC
- Q3 pad 2: Net-(J3-Pin_2) -> GND
- Q3 pad 3: VDC -> Net-(J3-Pin_2)
- Q4 pad 2: GND -> VDC
- Q5 pad 2: Net-(J3-Pin_3) -> GND
- Q5 pad 3: VDC -> Net-(J3-Pin_3)
- Q6 pad 2: GND -> VDC
- R1 pad 1: +3.3V -> /C2CK
- R1 pad 2: /C2CK -> +3.3V
Routing:
- net VDC: track 39.1 -> 43.3 mm
- net /COM_B: track 14.9 -> 12.8 mm
- net Net-(J3-Pin_2): track 14.4 -> 12.7 mm
- net +3.3V: track 14.7 -> 13.3 mm, vias 2 -> 1
- net Net-(J3-Pin_1): track 13.1 -> 11.9 mm
- net Net-(J3-Pin_3): track 15.5 -> 14.4 mm
- net /MUX_C: track 14.3 -> 13.2 mm
- net GND: track 7.64 -> 7.16 mm, vias 15 -> 18
Other:
- outline, holes or cut-outs redrawn
- board text added: "G 3V CK CD"
- board text removed: "G CK 3V D"
