File: pcb_blheli_s.kicad_sch (KiCad schematic)
At the start: 23 parts, among them IC1 EFM8BB21F16G-C-QFN20, IC2 REG113NA-3.3_250, J1 Conn_01x03_Pin, J2 Conn_01x04_Pin, J3 Conn_01x03_Socket, Q1 DMN2058U, Q2 DMN2058U, Q3 DMN2058U, Q4 DMN2058U, Q5 DMN2058U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

Commit message: Updated schematics
Parts:
- added J4: Conn_01x03_Pin, Connector_PinHeader_2.00mm:PinHeader_1x03_P2.00mm_Vertical, symbol Connector:Conn_01x03_Pin
- added R10, R11, R9: 2K2, Resistor_SMD:R_0603_1608Metric, symbol Device:R_Small
- J3: footprint Connector_PinHeader_1.27mm:PinHeader_1x03_P1.27mm_Vertical -> Connector_PinHeader_2.00mm:PinHeader_1x03_P2.00mm_Vertical
Connections:
- net GND: now also Q2.2 (S), Q4.2 (S), Q6.2 (S), J4.3 (Pin_3), R10.1, R11.1, R9.1; no longer Q1.2 (S), Q3.2 (S), Q5.2 (S)
- net MUX_A: now also R9.2
- net MUX_B: now also R10.2
- net MUX_C: now also R11.2
- net VDC: now also Q1.3 (D), Q3.3 (D), Q5.3 (D); no longer Q2.2 (S), Q4.2 (S), Q6.2 (S)
- net at J3.2 (Pin_2), Q4.3 (D), R5.1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: now also Q3.2 (S); no longer Q3.3 (D)
- net at J3.1 (Pin_1), Q2.3 (D), R3.1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: now also Q1.2 (S); no longer Q1.3 (D)
- net at J3.3 (Pin_3), Q6.3 (D), R7.1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: now also Q5.2 (S); no longer Q5.3 (D)
- net RX0: now reaches IC1.17 (P0.5), R2.1
- net RX0: now also J4.2 (Pin_2)
- net BL_TX2 renamed TX0
- net TX0: now also J4.1 (Pin_1)
Other:
- moved on the sheet: Q1, Q2, Q3, Q4, Q5, Q6, R4, R6, R8

Commit message: Ordered rev2
Parts:
- removed Q2, Q4, Q6: DMN2058U, Package_TO_SOT_SMD:SOT-23, symbol Transistor_FET:DMN2058U
- added Q2, Q4, Q6: IRLML2244TRPBF, footprint_blheli:SOT95P237X112-3N, symbol lib_blheli:IRLML2244TRPBF
Connections:
- net +3.3V: now also J2.2 (Pin_2), R1.2; no longer J2.3 (Pin_3), R1.1
- net C2CK: now also J2.3 (Pin_3), R1.1; no longer J2.2 (Pin_2), R1.2
- net COM_A: now also Q2.1 (G)
- net COM_B: now also Q4.1 (G)
- net COM_C: now also Q6.1 (G)
- net GND: now also Q1.2 (S), Q3.2 (S), Q5.2 (S)
- net VDC: now also Q2.2 (S), Q4.2 (S), Q6.2 (S); no longer Q1.3 (D), Q3.3 (D), Q5.3 (D)
- net at J3.2 (Pin_2), R5.1, R6.2: now also Q3.3 (D), Q4.3 (D); no longer Q3.2 (S)
- net at J3.1 (Pin_1), R3.1, R4.2: now also Q1.3 (D), Q2.3 (D); no longer Q1.2 (S)
- net at J3.3 (Pin_3), R7.1, R8.2: now also Q5.3 (D), Q6.3 (D); no longer Q5.2 (S)
Other:
- note added: "DO NOT POPULATE"
- moved on the sheet: J1, J2, J4, Q1, Q3, Q5, R1
